File: hardware/vanchor-helm.kicad_sch (KiCad schematic)
At the start: 0 parts

Commit message: feat: all five schematic sheets + root, ERC 0 errors, netlist gate PASS
- netlist-style sheets generated from python net specs (sheets/*.py)
- 94 nets / 334 pins; key-net pin-count check in scripts/check_nets.py
- ERC waivers documented in hardware/ERC-notes.md

Co-Authored-By: Claude Fable 5 <noreply@anthropic.com>
Other:
- added sheet mcu (mcu.kicad_sch)
- added sheet pi (pi.kicad_sch)
- added sheet power (power.kicad_sch)
- added sheet servo (servo.kicad_sch)
- added sheet thrust (thrust.kicad_sch)
- note added: "Vanchor Helm Board — sheet index\n1 power: battery in, protection, 5V/12V rails\n2 pi: Pi carrier, UARTs, I2C, display/fan power\n3 mcu: Pico 2 controller\n4 thrust: external 1500W controller hijack + contactor\n5 servo: IBT-2 header + AS5600 encoder"
Changed lines of the file:
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@@
     (rev "A")
     (company "vanchor-ng")
+    (comment 1 "Pi 4/5 carrier + Pico 2: trolling motor thrust (digipot hijack) + AS5600 servo")
+    (comment 2 "12-48V in; 1500W path stays off-board (external controller + contactor)")
+  )
+  (text "Vanchor Helm Board — sheet index\\n1 power: battery in, protection, 5V/12V rails\\n2 pi: Pi carrier, UARTs, I2C, display/fan power\\n3 mcu: Pico 2 controller\\n4 thrust: external 1500W controller hijack + contactor\\n5 servo: IBT-2 header + AS5600 encoder"
+    (exclude_from_sim no)
+    (at 30 40 0)
+    (effects (font (size 2.5 2.5)) (justify left bottom))
+    (uuid "a0000000-0000-4000-8000-00000000t001")
+  )
+  (sheet
+    (at 40 60)
+    (size 50 25)
+    (fields_autoplaced yes)
+    (stroke (width 0.1524) (type solid))
+    (fill (color 0 0 0 0.0000))
+    (property "Sheetname" "power"
+      (at 40 59.2 0)
+      (effects (font (size 1.27 1.27)) (justify left bottom))
+    )
+    (property "Sheetfile" "power.kicad_sch"
+      (at 40 85.6 0)
+      (effects (font (size 1.27 1.27)) (justify left top) (hide yes))
+    )
+    (instances (project "vanchor-helm" (path "/a0000000-0000-4000-8000-000000000001" (page "2"))))
+  )
+  (sheet
+    (at 110 60)
+    (size 50 25)
+    (fields_autoplaced yes)
+    (stroke (width 0.1524) (type solid))
+    (fill (color 0 0 0 0.0000))
+    (property "Sheetname" "pi"
+      (at 110 59.2 0)
+      (effects (font (size 1.27 1.27)) (justify left bottom))
+    )
+    (property "Sheetfile" "pi.kicad_sch"
+      (at 110 85.6 0)
+      (effects (font (size 1.27 1.27)) (justify left top) (hide yes))
+    )
+    (instances (project "vanchor-helm" (path "/a0000000-0000-4000-8000-000000000001" (page "3"))))
+  )
+  (sheet
+    (at 180 60)
+    (size 50 25)
+    (fields_autoplaced yes)
+    (stroke (width 0.1524) (type solid))
+    (fill (color 0 0 0 0.0000))
+    (property "Sheetname" "mcu"
+      (at 180 59.2 0)
+      (effects (font (size 1.27 1.27)) (justify left bottom))
+    )
+    (property "Sheetfile" "mcu.kicad_sch"
+      (at 180 85.6 0)
+      (effects (font (size 1.27 1.27)) (justify left top) (hide yes))
+    )
+    (instances (project "vanchor-helm" (path "/a0000000-0000-4000-8000-000000000001" (page "4"))))
+  )
+  (sheet
+    (at 250 60)
+    (size 50 25)
+    (fields_autoplaced yes)
+    (stroke (width 0.1524) (type solid))
+    (fill (color 0 0 0 0.0000))
+    (property "Sheetname" "thrust"
+      (at 250 59.2 0)
+      (effects (font (size 1.27 1.27)) (justify left bottom))
+    )
+    (property "Sheetfile" "thrust.kicad_sch"
+      (at 250 85.6 0)
+      (effects (font (size 1.27 1.27)) (justify left top) (hide yes))
+    )
+    (instances (project "vanchor-helm" (path "/a0000000-0000-4000-8000-000000000001" (page "5"))))
+  )
+  (sheet
+    (at 320 60)
+    (size 50 25)
+    (fields_autoplaced yes)
+    (stroke (width 0.1524) (type solid))
+    (fill (color 0 0 0 0.0000))
+    (property "Sheetname" "servo"
+      (at 320 59.2 0)
+      (effects (font (size 1.27 1.27)) (justify left bottom))
+    )
+    (property "Sheetfile" "servo.kicad_sch"
+      (at 320 85.6 0)
+      (effects (font (size 1.27 1.27)) (justify left top) (hide yes))
+    )
+    (instances (project "vanchor-helm" (path "/a0000000-0000-4000-8000-000000000001" (page "6"))))
   )
   (sheet_instances

Commit message: fix: F2 footprint MF-RG300 (was oversized RG400, body offset); feat: readable 2-page schematic (carrier/control merged specs)
Co-Authored-By: Claude Fable 5 <noreply@anthropic.com>
Other:
- sheet mcu renamed control
- sheet power renamed carrier
- removed sheet pi
- removed sheet servo
- removed sheet thrust
- sheet carrier: file power.kicad_sch -> carrier.kicad_sch
- sheet control: file mcu.kicad_sch -> control.kicad_sch
- note added: "1 carrier: 12V in, protection, 5V buck header, Orange Pi Zero 3 ribbon header, UART/I2C JSTs"
- note added: "2 control: Pico 2, external thrust-driver interface (J13), BTN8982 servo bridge, AS5600"
- note added: "Vanchor Helm Board - sheet index"
- note removed: "Vanchor Helm Board — sheet index\n1 power: battery in, protection, 5V/12V rails\n2 pi: Pi carrier, UARTs, I2C, display/fan power\n3 mcu: Pico 2 controller\n4 thrust: external 1500W controller hijack + contactor\n5 servo: IBT-2 header + AS5600 encoder"
Changed lines of the file:
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@@
   (title_block
     (title "Vanchor Helm Board")
-    (date "2026-07-01")
-    (rev "A")
+    (date "2026-07-02")
+    (rev "v4.1")
     (company "vanchor-ng")
-    (comment 1 "Pi 4/5 carrier + Pico 2: trolling motor thrust (digipot hijack) + AS5600 servo")
-    (comment 2 "12-48V in; 1500W path stays off-board (external controller + contactor)")
+    (comment 1 "Orange Pi Zero 3 (IDC ribbon) + Pico 2; external IBT-2 thrust driver; on-board servo bridge")
+    (comment 2 "12V battery only; 5V from generic buck module on J14")
   )
-  (text "Vanchor Helm Board — sheet index\\n1 power: battery in, protection, 5V/12V rails\\n2 pi: Pi carrier, UARTs, I2C, display/fan power\\n3 mcu: Pico 2 controller\\n4 thrust: external 1500W controller hijack + contactor\\n5 servo: IBT-2 header + AS5600 encoder"
+  (text "Vanchor Helm Board - sheet index"
     (exclude_from_sim no)
-    (at 30 40 0)
-    (effects (font (size 2.5 2.5)) (justify left bottom))
+    (at 30 32 0)
+    (effects (font (size 3 3)) (justify left bottom))
     (uuid "a0000000-0000-4000-8000-00000000t001")
   )
+  (text "1  carrier: 12V in, protection, 5V buck header, Orange Pi Zero 3 ribbon header, UART/I2C JSTs"
+    (exclude_from_sim no)
+    (at 30 42 0)
+    (effects (font (size 2 2)) (justify left bottom))
+    (uuid "a0000000-0000-4000-8000-00000000t002")
+  )
+  (text "2  control: Pico 2, external thrust-driver interface (J13), BTN8982 servo bridge, AS5600"
+    (exclude_from_sim no)
+    (at 30 50 0)
+    (effects (font (size 2 2)) (justify left bottom))
+    (uuid "a0000000-0000-4000-8000-00000000t003")
+  )
   (sheet
-    (at 40 60)
-    (size 50 25)
+    (at 40 70)
+    (size 70 30)
     (fields_autoplaced yes)
     (stroke (width 0.1524) (type solid))
     (fill (color 0 0 0 0.0000))
-    (property "Sheetname" "power"
-      (at 40 59.2 0)
+    (property "Sheetname" "carrier"
+      (at 40 69.2 0)
       (effects (font (size 1.27 1.27)) (justify left bottom))
     )
-    (property "Sheetfile" "power.kicad_sch"
-      (at 40 85.6 0)
+    (property "Sheetfile" "carrier.kicad_sch"
+      (at 40 100.6 0)
       (effects (font (size 1.27 1.27)) (justify left top) (hide yes))
     )
@@
   )
   (sheet
-    (at 110 60)
-    (size 50 25)
+    (at 130 70)
+    (size 70 30)
     (fields_autoplaced yes)
     (stroke (width 0.1524) (type solid))
     (fill (color 0 0 0 0.0000))
-    (property "Sheetname" "pi"
-      (at 110 59.2 0)
+    (property "Sheetname" "control"
+      (at 130 69.2 0)
       (effects (font (size 1.27 1.27)) (justify left bottom))
     )
-    (property "Sheetfile" "pi.kicad_sch"
-      (at 110 85.6 0)
+    (property "Sheetfile" "control.kicad_sch"
+      (at 130 100.6 0)
       (effects (font (size 1.27 1.27)) (justify left top) (hide yes))
     )
     (instances (project "vanchor-helm" (path "/a0000000-0000-4000-8000-000000000001" (page "3"))))
   )
-  (sheet
-    (at 180 60)
-    (size 50 25)
-    (fields_autoplaced yes)
-    (stroke (width 0.1524) (type solid))
-    (fill (color 0 0 0 0.0000))
-    (property "Sheetname" "mcu"
-      (at 180 59.2 0)
-      (effects (font (size 1.27 1.27)) (justify left bottom))
-    )
-    (property "Sheetfile" "mcu.kicad_sch"
-      (at 180 85.6 0)
-      (effects (font (size 1.27 1.27)) (justify left top) (hide yes))
-    )
-    (instances (project "vanchor-helm" (path "/a0000000-0000-4000-8000-000000000001" (page "4"))))
-  )
-  (sheet
-    (at 250 60)
-    (size 50 25)
-    (fields_autoplaced yes)
-    (stroke (width 0.1524) (type solid))
-    (fill (color 0 0 0 0.0000))
-    (property "Sheetname" "thrust"
-      (at 250 59.2 0)
-      (effects (font (size 1.27 1.27)) (justify left bottom))
-    )
-    (property "Sheetfile" "thrust.kicad_sch"
-      (at 250 85.6 0)
-      (effects (font (size 1.27 1.27)) (justify left top) (hide yes))
-    )
-    (instances (project "vanchor-helm" (path "/a0000000-0000-4000-8000-000000000001" (page "5"))))
-  )
-  (sheet
-    (at 320 60)
-    (size 50 25)
-    (fields_autoplaced yes)
-    (stroke (width 0.1524) (type solid))
-    (fill (color 0 0 0 0.0000))
-    (property "Sheetname" "servo"
-      (at 320 59.2 0)
-      (effects (font (size 1.27 1.27)) (justify left bottom))
-    )
-    (property "Sheetfile" "servo.kicad_sch"
-      (at 320 85.6 0)
-      (effects (font (size 1.27 1.27)) (justify left top) (hide yes))
-    )
-    (instances (project "vanchor-helm" (path "/a0000000-0000-4000-8000-000000000001" (page "6"))))
-  )
-  (sheet_instances
-    (path "/" (page "1"))
-  )
+  (sheet_instances (path "/" (page "1")))
 )
