File: boards/thrust-driver/vanchor-thrust.kicad_pcb (KiCad board)
At the start: 2 copper layers, 95 x 75 mm, 27 parts, among them J1 HELM J13 1:1, J2 LUG BATT+, J3 LUG BATT-, J4 LUG MOT A, J5 LUG MOT B, U1 BTN8982TA, U2 BTN8982TA, U3 BTN8982TA, U4 BTN8982TA

Commit message: feat(thrust-driver): NMEA2000 smart-node provision — DNP Pico 2 + CAN/N2K connectors, board 95x92
Unpopulated through-hole provision to run the bridge as a standalone N2K
node: U5 Pico 2 (GP12-15 parallel to J1 drive nets, GP26/27 ADC sense via
R12/R13 1k, GP18/19 CAN), U6 SIP-3 5V reg from VBAT, J6 transceiver
header (3V3/GND/TX/RX), J7 N2K V+/GND/SHIELD with 0R power-tap/shield
options. Board grew 75->92mm; existing routing untouched; DRC 0 errors /
0 unconnected (solder-lane mask apertures set to ignore by design).

Co-Authored-By: Claude Fable 5 <noreply@anthropic.com>
Parts:
- added H3: MountingHole, MountingHole_3.2mm_M3, F.Cu at (88.0, 28.0)
- added H4: MountingHole, MountingHole_3.2mm_M3, F.Cu at (111.5, 91.0)
- added J6: CAN XCVR, PinHeader_1x04_P2.54mm_Vertical, F.Cu at (95.0, 102.2)
- added J7: NMEA2000 PWR, JST_XH_B3B-XH-A_1x03_P2.50mm_Vertical, F.Cu at (106.5, 103.0)
- added R10: 0R DNP, R_0805_2012Metric, F.Cu at (101.0, 106.5)
- added R11: 0R DNP, R_0805_2012Metric, F.Cu at (104.8, 109.3)
- added R12: 1k DNP, R_0805_2012Metric, F.Cu at (42.8, 75.0)
- added R13: 1k DNP, R_0805_2012Metric, F.Cu at (46.2, 78.2)
- added U5: Pico 2 (DNP), RaspberryPi_Pico_TH_SWD, F.Cu at (36.2, 109.9)
- added U6: R-78E5.0 (DNP), Converter_DCDC_TRACO_TSR-1_THT, F.Cu at (24.4, 100.3)
- moved D1 5.06 mm to (40.2, 83.6)
Routing:
- net VBAT: track 181.1 -> 343.0 mm, vias 4 -> 5
- net R_EN: track 55.8 -> 175.2 mm
- net RPWM: track 51.8 -> 169.8 mm
- net L_EN: track 68.8 -> 186.6 mm
- net LPWM: track 62.2 -> 178.9 mm
- net +3V3: track 0.00 -> 58.7 mm
- net CAN_RX: track 0.00 -> 38.4 mm
- net CAN_TX: track 0.00 -> 33.3 mm
- net +5V: track 40.2 -> 71.5 mm, vias 0 -> 1
- net R_ADC: track 0.00 -> 29.3 mm, vias 0 -> 1
- net L_ADC: track 0.00 -> 25.9 mm, vias 0 -> 1
- net GND: track 78.4 -> 100.7 mm
- net N2K_SHLD: track 0.00 -> 16.4 mm
- net R_IS: track 66.3 -> 81.7 mm, vias 4 -> 6
- net N2K_VP: track 0.00 -> 11.9 mm
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Other:
- board size 95 x 75 mm -> 95 x 92 mm
- board text added: "3V3 GND TX RX"
- board text added: "5V REG"
- board text added: "CAN"
- board text added: "N2K PWR"
- board text added: "PICO 2 - N2K NODE OPTION (DNP)"
- board text added: "SMART NODE: FIT U5 U6 R12 R13 + CAN XCVR ON J6, LEAVE J1 OPEN"
- board text added: "V+ GND SH"
