File: boards/helm/vanchor-helm.kicad_pcb (KiCad board)
At the start: 2 copper layers, 125 x 95 mm, 63 parts, among them J1 OPI_Z3_26PIN, J10 AUX 5V (screen), J11 AS5600, J12 PICO UTIL, J13 THRUST DRV, J16 BATT 12V, J2 OPI_BREAKOUT, J22 SERVO MOTOR, J3 UART5 ttyAS5, J4 UART2 ttyAS2, J8 I2C3 spare, J9 FAN 5V, Q1 IRF9540N, U1 Pico 2, U5 XL4015 5A, U7 BTN8982TA, U8 BTN8982TA

Commit message: feat(helm): J2 doubles as Raspberry Pi port (classic 26-pin positions), silk + docs
The PI26 net map already follows the classic RPi 26-pin layout, so a
Raspberry Pi (40-pin header pins 1-26) drops onto J2 via the same 26-way
IDC ribbon: power, Pico I2C link (SDA1/SCL1), console UART (TXD0/RXD0),
SPI and SWD/RUN GPIOs all line up. Fit one SBC only; J4 'UART2' JST is
bit-bang-only on an RPi (pins 11/13 are plain GPIOs there).

Co-Authored-By: Claude Fable 5 <noreply@anthropic.com>
Parts:
- J2: value OPI_BREAKOUT -> SBC2_OPI_RPI26
Other:
- board text added: "SBC2: OPI Z3 / RPI PINS 1-26 (FIT ONE SBC)"
Changed lines of the file:
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@@
 			)
 		)
-		(property "Value" "OPI_BREAKOUT"
+		(property "Value" "SBC2_OPI_RPI26"
 			(at 1.27 32.86 90)
 			(layer "F.Fab")
@@
 			)
 		)
+	)
+	(gr_text "1"
+		(at 32.799999 65.9 0)
+		(layer "F.SilkS")
+		(effects
+			(font
+				(size 0.8 0.8)
+				(thickness 0.15)
+			)
+		)
+	)
+	(gr_text "SBC2: OPI Z3 / RPI PINS 1-26 (FIT ONE SBC)"
+		(at 50 61.3 0)
+		(layer "F.SilkS")
+		(effects
+			(font
+				(size 0.8 0.8)
+				(thickness 0.15)
+			)
+		)

Commit message: feat(helm): NMEA2000/CAN provision — J5 power/shield connector, VIN tap, CAN-on-J12 docs
CAN rides the Pico 2 (can2040 on GP18/GP19); a 3.3V transceiver module
(Waveshare SN65HVD230) plugs J12 pins 1/8/6/7. New J5 XH-3 lands the N2K
drop cable's V+/GND/SHIELD; R41 (0R DNP) optionally powers the backbone
from VIN, R42 (0R DNP) bonds shield to GND. DRC 0/0.

Co-Authored-By: Claude Fable 5 <noreply@anthropic.com>
Parts:
- added J5: NMEA2000 PWR, JST_XH_B3B-XH-A_1x03_P2.50mm_Vertical, F.Cu at (24.5, 34.5)
- added R41: 0R DNP, R_0805_2012Metric, F.Cu at (34.5, 39.5)
- added R42: 0R DNP, R_0805_2012Metric, F.Cu at (23.2, 41.0)
Routing:
- net N2K_VP: track 0.00 -> 15.3 mm, vias 0 -> 1
- net N2K_SHLD: track 0.00 -> 8.46 mm
- net VIN: track 286.4 -> 292.9 mm
- net GND: track 680.2 -> 682.4 mm, vias 57 -> 58
Other:
- board text added: "CAN XCVR ON J12: 3V3=1 GND=8 TX=6 RX=7"
- board text added: "NMEA2000"
- board text added: "V+ - SH"

Commit message: feat(helm): steering-zero hall sensor input — J9 grows to 1x3 (5V/GND/SIG), 10k pullup + RC into Pico GP0
Open-collector hall switch (A3144 class) sees a magnet at servo center;
GP0 reads it (also broken out on J12.2; UART0 fallback = GP16/GP1).
Pour-redundant freerouted GND returns near J9/J10 removed. DRC 0/0.

Co-Authored-By: Claude Fable 5 <noreply@anthropic.com>
Parts:
- added C24: 100n, C_0805_2012Metric, F.Cu at (134.0, 44.6)
- added R22: 10k, R_0805_2012Metric, F.Cu at (134.0, 42.3)
- added R23: 1k, R_0805_2012Metric, F.Cu at (134.0, 40.0)
- J9: value FAN 5V -> FAN + HALL; footprint PinHeader_1x02_P2.54mm_Vertical -> PinHeader_1x03_P2.54mm_Vertical
Routing:
- net +3V3: track 258.8 -> 333.8 mm, vias 2 -> 3
- net GND: track 682.4 -> 654.9 mm, vias 58 -> 59
- net HALL_ZERO: track 0.00 -> 14.1 mm
- net PICO_GP0: track 117.2 -> 129.1 mm
Other:
- board text added: "5V G S"
- board text added: "FAN+HALL"
- board text removed: "FAN"

Commit message: fix(helm): F2 polyfuse sits straight — custom MF-R250 footprint with in-line 5.1mm pads (KiCad's Bourns fps are stagger-lead), pour-redundant GND returns cleared. DRC 0/0
Co-Authored-By: Claude Fable 5 <noreply@anthropic.com>
Parts:
- F2: footprint Fuse_Bourns_MF-RG300 -> MF-R250_Straight
Routing:
- net GND: track 654.9 -> 638.9 mm
- net DISP_5V: track 19.6 -> 18.4 mm
Changed lines of the file:
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@@
 		)
 	)
+	(footprint "MF-R250_Straight"
+		(layer "F.Cu")
+		(at 134.45 52.4)
+		(descr "Bourns MF-R250 polyfuse, straight radial leads, 5.1mm pitch")
+		(property "Reference" "F2"
+			(at 2.55 -3.4 0)
+			(layer "F.SilkS")
+			(effects
+				(font
+					(size 1 1)
+					(thickness 0.15)
+				)
+			)
+		)
+		(property "Value" "MF-R250 2.5A"
+			(at 2.55 3.4 0)
+			(layer "F.Fab")
+			(effects
+				(font
+					(size 1 1)
+					(thickness 0.15)
+				)
+			)
+		)
+		(property "Datasheet" ""
+			(at 0 0 0)
+			(layer "F.Fab")
+			(hide yes)
+			(effects
+				(font
+					(size 1.27 1.27)
+				)
+			)
+		)
+		(property "Description" ""
+			(at 0 0 0)
+			(layer "F.Fab")
+			(hide yes)
+			(effects
+				(font
+					(size 1.27 1.27)
+				)
+			)
+		)
+		(attr through_hole)
+		(duplicate_pad_numbers_are_jumpers no)
+		(fp_line
+			(start -2 -2.3)
+			(end 7.1 -2.3)
+			(stroke
+				(width 0.12)
+				(type solid)
+			)
+			(layer "F.SilkS")
+		)
+		(fp_line
+			(start -2 2.3)
+			(end -2 -2.3)
+			(stroke
+				(width 0.12)
+				(type solid)
+			)
+			(layer "F.SilkS")
+		)
+		(fp_line
+			(start 7.1 -2.3)
+			(end 7.1 2.3)
+			(stroke
+				(width 0.12)
+				(type solid)
+			)
+			(layer "F.SilkS")
+		)
+		(fp_line
+			(start 7.1 2.3)
+			(end -2 2.3)
+			(stroke
+				(width 0.12)
+				(type solid)
+			)
+			(layer "F.SilkS")
+		)
+		(fp_rect
+			(start -2.3 -2.6)
+			(end 7.4 2.6)
+			(stroke
+				(width 0.05)
+				(type solid)
+			)
+			(fill no)
+			(layer "F.CrtYd")
+		)
+		(fp_line
+			(start -2 -2.3)
+			(end 7.1 -2.3)
+			(stroke
+				(width 0.1)
+				(type solid)
+			)
+			(layer "F.Fab")
+		)
+		(fp_line
+			(start -2 2.3)
+			(end -2 -2.3)
+			(stroke
+				(width 0.1)
+				(type solid)
+			)
+			(layer "F.Fab")
+		)
+		(fp_line
+			(start 7.1 -2.3)
+			(end 7.1 2.3)
+			(stroke
+				(width 0.1)
+				(type solid)
+			)
+			(layer "F.Fab")
+		)
+		(fp_line
+			(start 7.1 2.3)
+			(end -2 2.3)
+			(stroke
+				(width 0.1)
+				(type solid)
+			)
+			(layer "F.Fab")
+		)
+		(pad "1" thru_hole circle
+			(at 0 0)
+			(size 1.8 1.8)
+			(drill 1)
+			(layers "*.Cu" "*.Mask")
+			(remove_unused_layers no)
+			(net "+5V")
+		)
+		(pad "2" thru_hole circle
+			(at 5.1 0)
+			(size 1.8 1.8)
+			(drill 1)
+			(layers "*.Cu" "*.Mask")
+			(remove_unused_layers no)
+			(net "DISP_5V")
+		)
+		(embedded_fonts no)
+	)
 	(footprint "R_Axial_DIN0207_L6.3mm_D2.5mm_P10.16mm_Horizontal"
 		(layer "F.Cu")
@@
 		)
 	)
-	(footprint "Fuse_Bourns_MF-RG300"
-		(layer "F.Cu")
-		(at 134.45 52.4)
-		(descr "PTC Resettable Fuse, Ihold = 3.0A, Itrip=5.1A, http://www.bourns.com/docs/Product-Datasheets/mfrg.pdf")
-		(tags "ptc resettable fuse polyfuse THT")
-		(property "Reference" "F2"
-			(at 2.55 -1.9 0)
-			(layer "F.SilkS")
-			(effects
-				(font
-					(size 1 1)
-					(thickness 0.15)
-				)
-			)
-		)
-		(property "Value" "MF-R250 2.5A"
-			(at 2.55 3.1 0)
-			(layer "F.Fab")
-			(effects
-				(font
-					(size 1 1)
-					(thickness 0.15)
-				)
-			)
-		)
-		(property "Datasheet" ""
-			(at 0 0 0)
-			(layer "F.Fab")
-			(hide yes)
-			(effects
-				(font
-					(size 1.27 1.27)
-				)
-			)
-		)
-		(property "Description" ""
-			(at 0 0 0)
-			(layer "F.Fab")
-			(hide yes)
-			(effects
-				(font
-					(size 1.27 1.27)
-				)
-			)
-		)
-		(attr through_hole)
-		(duplicate_pad_numbers_are_jumpers no)
-		(fp_line
-			(start -1.1 -1)
-			(end -0.838 -1)
-			(stroke
-				(width 0.12)
-				(type solid)
-			)
-			(layer "F.SilkS")
-		)
-		(fp_line
-			(start -1.1 -0.702)
-			(end -1.1 -1)
-			(stroke
-				(width 0.12)
-				(type solid)
-			)
-			(layer "F.SilkS")
-		)
-		(fp_line
-			(start -1.1 2.2)
-			(end -1.1 0.702)
-			(stroke
-				(width 0.12)
-				(type solid)
-			)
-			(layer "F.SilkS")
-		)
-		(fp_line
-			(start 0.838 -1)
-			(end 6.2 -1)
-			(stroke
-				(width 0.12)
-				(type solid)
-			)
-			(layer "F.SilkS")
-		)
-		(fp_line
-			(start 4.262 2.2)
-			(end -1.1 2.2)
-			(stroke
-				(width 0.12)
-				(type solid)
-			)
-			(layer "F.SilkS")
-		)
-		(fp_line
-			(start 6.2 -1)
-			(end 6.2 0.498)
-			(stroke
-				(width 0.12)
-				(type solid)
-			)
-			(layer "F.SilkS")
-		)
-		(fp_line
-			(start 6.2 1.902)
-			(end 6.2 2.2)
-			(stroke
-				(width 0.12)
-				(type solid)
-			)
-			(layer "F.SilkS")
-		)
-		(fp_line
-			(start 6.2 2.2)
-			(end 5.938 2.2)
-			(stroke
-				(width 0.12)
-				(type solid)
-			)
-			(layer "F.SilkS")
-		)
-		(fp_rect
-			(start -1.25 -1.15)
-			(end 6.35 2.35)
-			(stroke
-				(width 0.05)
-				(type solid)
-			)
-			(fill no)
-			(layer "F.CrtYd")
-		)
-		(fp_rect
-			(start -1 -0.9)
-			(end 6.1 2.1)
-			(stroke
-				(width 0.1)
-				(type solid)
-			)
-			(fill no)
-			(layer "F.Fab")
-		)
-		(fp_text user "${REFERENCE}"
-			(at 2.55 0.6 0)
-			(layer "F.Fab")
-			(effects
-				(font
-					(size 1 1)
-					(thickness 0.15)
-				)
-			)
-		)
-		(pad "1" thru_hole circle
-			(at 0 0)
-			(size 2.01 2.01)
-			(drill 1.01)
-			(layers "*.Cu" "*.Mask")
-			(remove_unused_layers no)
-			(net "+5V")
-		)
-		(pad "2" thru_hole circle
-			(at 5.1 1.2)
-			(size 2.01 2.01)
-			(drill 1.01)
-			(layers "*.Cu" "*.Mask")
-			(remove_unused_layers no)
-			(net "DISP_5V")
-		)
-		(embedded_fonts no)
-		(model "${KICAD9_3DMODEL_DIR}/Fuse.3dshapes/Fuse_Bourns_MF-RG300.step"
-			(offset
-				(xyz 0 0 0)
-			)
-			(scale
-				(xyz 1 1 1)
-			)
-			(rotate
-				(xyz 0 0 0)
-			)
-		)
-	)
 	(footprint "TO-220-3_Vertical"
 		(layer "F.Cu")
@@
 	)
 	(segment
-		(start 137 62.5)
-		(end 137 53.4453)
-		(width 1.5)
-		(layer "B.Cu")
-		(net "GND")
-	)
-	(segment
 		(start 66.7452 61.5831)
 		(end 66.7452 53.3348)
@@
 	)
 	(segment
-		(start 138.265 52.1803)
-		(end 138.265 47)
-		(width 1.5)
-		(layer "B.Cu")
-		(net "GND")
-	)
-	(segment
 		(start 31.3179 80.1071)
 		(end 31.3179 69.4844)
@@
 	)
 	(segment
-		(start 137 53.4453)
-		(end 138.265 52.1803)
-		(width 1.5)
-		(layer "B.Cu")
-		(net "GND")
-	)
-	(segment
 		(start 64.48 76.04)
 		(end 62.7541 77.7659)
@@
 	(segment
 		(start 139.55 38.325)
-		(end 139.55 53.6)
+		(end 139.55 52.4)
 		(width 0.3)
 		(layer "B.Cu")

Commit message: fix(helm): R41/R42 N2K option links are now hand-solderable THT vertical axials (were 0805); R41.2 lands directly in the VIN trunk
Co-Authored-By: Claude Fable 5 <noreply@anthropic.com>
Parts:
- R41, R42: footprint R_0805_2012Metric -> R_Axial_DIN0207_L6.3mm_D2.5mm_P2.54mm_Vertical
- moved R42 0.98 mm to (23.3, 42.0), turned to 90 degrees
- moved R41 0.91 mm to (33.6, 39.5), turned to 180 degrees
Routing:
- net VIN: track 292.9 -> 286.4 mm
- net GND: track 638.9 -> 644.2 mm
- net N2K_SHLD: track 8.46 -> 9.72 mm
