File: boards/helm/carrier.kicad_sch (KiCad schematic)
At the start: 25 parts, among them J1 OPI_Z3_26PIN, J10 AUX 5V (screen), J16 BATT 12V, J2 SBC2_OPI_RPI26, J3 UART5 ttyAS5, J4 UART2 ttyAS2, J5 NMEA2000 PWR, J8 I2C3 spare, J9 FAN + HALL, Q1 IRF9540N, U5 XL4015 5A

Commit message: fix(helm): R41/R42 N2K option links are now hand-solderable THT vertical axials (were 0805); R41.2 lands directly in the VIN trunk
Co-Authored-By: Claude Fable 5 <noreply@anthropic.com>
Parts:
- R41, R42: footprint Resistor_SMD:R_0805_2012Metric -> Resistor_THT:R_Axial_DIN0207_L6.3mm_D2.5mm_P2.54mm_Vertical
Changed lines of the file:
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@@
     (property "Value" "0R DNP" (at 345.44 135.89 0)
       (effects (font (size 1.27 1.27))))
-    (property "Footprint" "Resistor_SMD:R_0805_2012Metric" (at 345.44 128.27 0)
+    (property "Footprint" "Resistor_THT:R_Axial_DIN0207_L6.3mm_D2.5mm_P2.54mm_Vertical" (at 345.44 128.27 0)
       (effects (font (size 1.27 1.27)) (hide yes)))
     (property "Datasheet" "" (at 345.44 128.27 0)
@@
     (property "Value" "0R DNP" (at 361.95 157.48 0)
       (effects (font (size 1.27 1.27))))
-    (property "Footprint" "Resistor_SMD:R_0805_2012Metric" (at 361.95 149.86 0)
+    (property "Footprint" "Resistor_THT:R_Axial_DIN0207_L6.3mm_D2.5mm_P2.54mm_Vertical" (at 361.95 149.86 0)
       (effects (font (size 1.27 1.27)) (hide yes)))
     (property "Datasheet" "" (at 361.95 149.86 0)

Commit message: feat(gen_sheet): drawn wires + power rails (WIRES/RAILS spec lists) with per-cluster label dedup; wire up power chain, VIN rail, N2K links, sense rails, SR/LED chains
Co-Authored-By: Claude Fable 5 <noreply@anthropic.com>
Connections:
- net DISP_5V is gone; now on net +5V: F2.2, J10.1 (Pin_1)
- net VIN_RAW is gone; now on net Q1_G: F1.2, Q1.2 (D)
Changed lines of the file:
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@@
     (instances (project "vanchor-helm" (path "/a0000000-0000-4000-8000-000000000001/c0000000-0000-4000-8000-000000000002" (reference "#FLG04") (unit 1))))
   )
+  (wire (pts (xy 39.37 69.85) (xy 91.44 69.85))
+    (stroke (width 0) (type default)))
+  (wire (pts (xy 99.06 69.85) (xy 152.4 69.85))
+    (stroke (width 0) (type default)))
+  (wire (pts (xy 152.4 69.85) (xy 152.4 64.77))
+    (stroke (width 0) (type default)))
+  (wire (pts (xy 294.64 129.54) (xy 341.63 129.54))
+    (stroke (width 0) (type default)))
+  (wire (pts (xy 341.63 129.54) (xy 341.63 128.27))
+    (stroke (width 0) (type default)))
+  (wire (pts (xy 294.64 134.62) (xy 358.14 134.62))
+    (stroke (width 0) (type default)))
+  (wire (pts (xy 358.14 134.62) (xy 358.14 149.86))
+    (stroke (width 0) (type default)))
+  (wire (pts (xy 373.38 214.63) (xy 364.49 214.63))
+    (stroke (width 0) (type default)))
+  (wire (pts (xy 364.49 214.63) (xy 364.49 245.11))
+    (stroke (width 0) (type default)))
+  (wire (pts (xy 152.4 74.93) (xy 152.4 87.63))
+    (stroke (width 0) (type default)))
+  (wire (pts (xy 271.78 69.85) (xy 271.78 87.63))
+    (stroke (width 0) (type default)))
+  (wire (pts (xy 326.39 69.85) (xy 326.39 87.63))
+    (stroke (width 0) (type default)))
+  (wire (pts (xy 370.84 69.85) (xy 370.84 87.63))
+    (stroke (width 0) (type default)))
+  (wire (pts (xy 152.4 87.63) (xy 370.84 87.63))
+    (stroke (width 0) (type default)))
+  (junction (at 152.4 87.63) (diameter 0) (color 0 0 0 0)
+)
+  (junction (at 271.78 87.63) (diameter 0) (color 0 0 0 0)
+)
+  (junction (at 326.39 87.63) (diameter 0) (color 0 0 0 0)
+)
+  (junction (at 370.84 87.63) (diameter 0) (color 0 0 0 0)
+)
   (global_label "N2K_VP" (shape passive) (at 294.64 129.54 180.0) (fields_autoplaced yes)
     (effects (font (size 1.27 1.27)) (justify right))
@@
       (effects (font (size 1.27 1.27)) (hide yes)))
   )
-  (global_label "N2K_VP" (shape passive) (at 341.63 128.27 180.0) (fields_autoplaced yes)
-    (effects (font (size 1.27 1.27)) (justify right))
-    (property "Intersheetrefs" "${INTERSHEET_REFS}" (at 341.63 128.27 0)
-      (effects (font (size 1.27 1.27)) (hide yes)))
-  )
   (global_label "VIN" (shape passive) (at 349.25 128.27 0.0) (fields_autoplaced yes)
     (effects (font (size 1.27 1.27)) (justify left))
@@
       (effects (font (size 1.27 1.27)) (hide yes)))
   )
-  (global_label "N2K_SHLD" (shape passive) (at 358.14 149.86 180.0) (fields_autoplaced yes)
-    (effects (font (size 1.27 1.27)) (justify right))
-    (property "Intersheetrefs" "${INTERSHEET_REFS}" (at 358.14 149.86 0)
-      (effects (font (size 1.27 1.27)) (hide yes)))
-  )
   (global_label "GND" (shape passive) (at 365.76 149.86 0.0) (fields_autoplaced yes)
     (effects (font (size 1.27 1.27)) (justify left))
@@
       (effects (font (size 1.27 1.27)) (hide yes)))
   )
-  (label "BATT_IN" (at 91.44 69.85 180.0) (fields_autoplaced yes)
-    (effects (font (size 1.27 1.27)) (justify right))
-  )
   (label "VIN_RAW" (at 99.06 69.85 0.0) (fields_autoplaced yes)
     (effects (font (size 1.27 1.27)) (justify left))
@@
     (effects (font (size 1.27 1.27)) (justify right))
   )
-  (label "VIN_RAW" (at 152.4 64.77 90.0) (fields_autoplaced yes)
-    (effects (font (size 1.27 1.27)) (justify left))
-  )
   (global_label "VIN" (shape passive) (at 152.4 74.93 270.0) (fields_autoplaced yes)
     (effects (font (size 1.27 1.27)) (justify left))
@@
     (effects (font (size 1.27 1.27)) (justify left))
   )
-  (global_label "VIN" (shape passive) (at 271.78 69.85 180.0) (fields_autoplaced yes)
-    (effects (font (size 1.27 1.27)) (justify right))
-    (property "Intersheetrefs" "${INTERSHEET_REFS}" (at 271.78 69.85 0)
-      (effects (font (size 1.27 1.27)) (hide yes)))
-  )
   (global_label "GND" (shape passive) (at 279.4 69.85 0.0) (fields_autoplaced yes)
     (effects (font (size 1.27 1.27)) (justify left))
@@
       (effects (font (size 1.27 1.27)) (hide yes)))
   )
-  (global_label "VIN" (shape passive) (at 326.39 69.85 180.0) (fields_autoplaced yes)
-    (effects (font (size 1.27 1.27)) (justify right))
-    (property "Intersheetrefs" "${INTERSHEET_REFS}" (at 326.39 69.85 0)
-      (effects (font (size 1.27 1.27)) (hide yes)))
-  )
   (global_label "GND" (shape passive) (at 334.01 69.85 0.0) (fields_autoplaced yes)
     (effects (font (size 1.27 1.27)) (justify left))
@@
       (effects (font (size 1.27 1.27)) (hide yes)))
   )
-  (global_label "VIN" (shape passive) (at 370.84 69.85 180.0) (fields_autoplaced yes)
-    (effects (font (size 1.27 1.27)) (justify right))
-    (property "Intersheetrefs" "${INTERSHEET_REFS}" (at 370.84 69.85 0)
-      (effects (font (size 1.27 1.27)) (hide yes)))
-  )
   (global_label "GND" (shape passive) (at 378.46 69.85 0.0) (fields_autoplaced yes)
     (effects (font (size 1.27 1.27)) (justify left))
@@
       (effects (font (size 1.27 1.27)) (hide yes)))
   )
-  (global_label "DISP_5V" (shape passive) (at 364.49 245.11 180.0) (fields_autoplaced yes)
-    (effects (font (size 1.27 1.27)) (justify right))
-    (property "Intersheetrefs" "${INTERSHEET_REFS}" (at 364.49 245.11 0)
-      (effects (font (size 1.27 1.27)) (hide yes)))
-  )
