File: boards/helm/carrier.kicad_sch (KiCad schematic)
At the start: 25 parts, among them J1 OPI_Z3_26PIN, J10 AUX 5V (screen), J16 BATT 12V, J2 SBC2_OPI_RPI26, J3 UART5 ttyAS5, J4 UART2 ttyAS2, J5 NMEA2000 PWR, J8 I2C3 spare, J9 FAN + HALL, Q1 IRF9540N, U5 XL4015 5A

Commit message: fix(schematics): visual QA pass — text collisions and wire-through-symbol
gen_sheet: BAT54S ref+value stack below the part (COM pin label owns the
space above — fixes D8/D10/D11/D14 overprinted refs); REF_POS per-part
ref override. Carrier: F1->Q1 drain wire enters from above instead of
through the FET symbol; Q1 ref moved clear. Control: R20/R21 spread so
their texts don't merge; D14 lifted off the VBAT wire; LED_STAT run
raised above the pico power flags. Driver: ADC wires lose their dead-end
spurs; CAN lanes dropped below the DNP value texts; D2 horizontal (label
was overprinting ref/value). HANDOFF: waive note for the 3 paralleled-OUT
ERC errors. Netlists verified identical on both boards.

Co-Authored-By: Claude Fable 5 <noreply@anthropic.com>
Claude-Session: https://claude.ai/code/session_011PT4Xv5KGhDdDc8nqJyMxJ
Connections:
- net Q1_G: no longer F1.2, Q1.2 (D)
- new net VIN_RAW: F1.2, Q1.2 (D)
Changed lines of the file:
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@@
   (symbol (lib_id "Transistor_FET:IRF9540N") (at 149.86 69.85 0) (unit 1)
     (exclude_from_sim no) (in_bom yes) (on_board yes) (dnp no)
-    (property "Reference" "Q1" (at 149.86 60.96 0)
+    (property "Reference" "Q1" (at 144 61.11 0)
       (effects (font (size 1.27 1.27))))
     (property "Value" "IRF9540N" (at 149.86 78.74 0)
@@
   (wire (pts (xy 39.37 69.85) (xy 91.44 69.85))
     (stroke (width 0) (type default)))
-  (wire (pts (xy 99.06 69.85) (xy 152.4 69.85))
+  (wire (pts (xy 99.06 69.85) (xy 99.06 57.15))
     (stroke (width 0) (type default)))
-  (wire (pts (xy 152.4 69.85) (xy 152.4 64.77))
+  (wire (pts (xy 99.06 57.15) (xy 152.54 57.15))
+    (stroke (width 0) (type default)))
+  (wire (pts (xy 152.54 57.15) (xy 152.4 57.15))
+    (stroke (width 0) (type default)))
+  (wire (pts (xy 152.4 57.15) (xy 152.4 64.77))
     (stroke (width 0) (type default)))
   (wire (pts (xy 294.64 129.54) (xy 341.63 129.54))
