File: boards/helm/control.kicad_sch (KiCad schematic)
At the start: 38 parts, among them J11 AS5600, J12 PICO UTIL, J13 THRUST DRV, J22 SERVO MOTOR, U1 Pico 2, U7 BTN8982TA, U8 BTN8982TA

Commit message: fix(schematics): visual QA pass — text collisions and wire-through-symbol
gen_sheet: BAT54S ref+value stack below the part (COM pin label owns the
space above — fixes D8/D10/D11/D14 overprinted refs); REF_POS per-part
ref override. Carrier: F1->Q1 drain wire enters from above instead of
through the FET symbol; Q1 ref moved clear. Control: R20/R21 spread so
their texts don't merge; D14 lifted off the VBAT wire; LED_STAT run
raised above the pico power flags. Driver: ADC wires lose their dead-end
spurs; CAN lanes dropped below the DNP value texts; D2 horizontal (label
was overprinting ref/value). HANDOFF: waive note for the 3 paralleled-OUT
ERC errors. Netlists verified identical on both boards.

Co-Authored-By: Claude Fable 5 <noreply@anthropic.com>
Claude-Session: https://claude.ai/code/session_011PT4Xv5KGhDdDc8nqJyMxJ
Other:
- moved on the sheet: D14, R20, R21
